File: pcb/ExtenderCoco.sch (EAGLE design)
At the start: 12 parts, among them X1 EXPANSION_PORT_COCO, X2 EXPANSION_PORT_COCOS, X3 EXPANSION_PORT_COCOM

Commit message: Cart port connector was too narrow...
Parts:
- added C1: (no value), rcl:CPOL-USE2-5
- X2: value EXPANSION_PORT_COCOS -> EXPANSION_PORT_COCOM; device coco:EXPANSION_PORT_COCOS -> coco:EXPANSION_PORT_COCOM
- X3: value EXPANSION_PORT_COCOM -> EXPANSION_PORT_COCOS; device coco:EXPANSION_PORT_COCOM -> coco:EXPANSION_PORT_COCOS
Connections:
- new net GND: C1.-
- new net VCC: C1.+
